File: 01_Logger/02_Modular_Logger/01_Electronics/01_Main_Unit/Battery_Charger.kicad_sch (KiCad schematic)
At the start: 52 parts, among them IC501 BQ24618, J501 Conn_01x02, J502 Conn_01x02_Female, K501 SISH101DN-T1-GE3, K502 SISH101DN-T1-GE3, K503 SiS412DN, K504 SiS412DN, K505 SISH101DN-T1-GE3

Commit message: update Electronics for Modular_Logger
Parts:
- R501: value 2 -> 100
- R522: value 348k -> 357k
