File: 01_Logger/02_Modular_Logger/01_Electronics/01_Main_Unit/MPU.kicad_sch (KiCad schematic)
At the start: 38 parts, among them J301 Conn_01x02, J302 Conn_02x04_Counter_Clockwise, J303 Conn_01x02, J304 Conn_02x02_Odd_Even, Q301 BSS138, SW301 SW_Push, U301 MAX16125WTEG00+T, U302 ESP32-S3-WROOM-1U, U303 DS3231MZ, Y301 Crystal

Commit message: update Electronics for Modular_Logger
Parts:
- added R703: 1M, Resistor_SMD:R_0603_1608Metric, symbol Device:R
- U301: symbol MAX6071ANT25_T:MAX16124/5 -> MAX6071ANT25_T:MAX16124/5
Connections:
- net GND: now also R703.2
- net LED_STATUS: now also R703.1
